File: project/ECAD/PCB-MachineThatDraws/PCB-MachineThatDraws.kicad_pcb (KiCad board)
At the start: 2 copper layers, 53.5 x 83 mm, 29 parts, among them J1 SD_Card_Device, J10 Conn_02x03_Odd_Even, J11 Conn_02x03_Odd_Even, J2 SDA/SCL/VCC/GND, J3 Switch, J4 Limit_Switch_X, J5 Moteur, J6 Moteur, J7 Barrel_Jack_Switch, J8 Screw_Terminal_01x02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

Commit message: pcb up
Parts:
- J10, J11: moved to F.Cu
- moved J11 5.19 mm to (112.0, 76.8)
- moved J10 5.03 mm to (129.5, 76.8)
